Commit message: Generate test vehicle

File: test/models/gazebo_ros_four_wheel_steering_test_vehicle/wheel.urdf.xacro (robot description, xacro)
@@ -13,5 +13,5 @@
       name="wheel"
       params="wheel_prefix parent_link *origin">
-    <link name="${wheel_prefix}_wheel_link">
+    <link name="${wheel_prefix}_wheel">
       <xacro:cylinder_primitive
           length="${wheel_length}"
@@ -26,8 +26,8 @@
     </link>
     <joint
-        name="${wheel_prefix}_wheel"
+        name="${wheel_prefix}_motor"
         type="continuous">
       <parent link="${parent_link}" />
-      <child link="${wheel_prefix}_wheel_link" />
+      <child link="${wheel_prefix}_wheel" />
       <xacro:insert_block name="origin" />
       <limit
