Commit message: Controllable geometry

File: test/models/gazebo_ros_four_wheel_steering_test_vehicle/model.urdf.xacro (robot description, xacro)
@@ -3,26 +3,31 @@
     name="gazebo_ros_four_wheel_steering_test_vehicle"
     xmlns:xacro="http://ros.org/wiki/xacro">
-  <xacro:include filename="$(arg xacro_prefix)/urdf/four_wheel_steering.urdf.xacro" />
-  <xacro:include filename="$(arg xacro_prefix)/urdf/inertia_tensors.urdf.xacro" />
-  <xacro:include filename="$(arg xacro_prefix)/urdf/primitives.urdf.xacro" />
+  <xacro:include filename="$(arg gazebo_ros_four_wheel_steering_prefix)/urdf/four_wheel_steering.urdf.xacro" />
+  <xacro:include filename="$(arg gazebo_ros_four_wheel_steering_prefix)/urdf/inertia_tensors.urdf.xacro" />
+  <xacro:include filename="$(arg gazebo_ros_four_wheel_steering_prefix)/urdf/primitives.urdf.xacro" />
   <xacro:include filename="wheel.urdf.xacro" />
   <xacro:property
-      name="wheel_track"
-      value="1.6" />
+      name="axle_width"
+      value="1.06" />
+  <xacro:property
+      name="axle_wheel_offset_y"
+      value="0.06" />
   <xacro:property
       name="wheel_base"
-      value="1.5" />
+      value="1.1" />
   <link name="chassis">
     <xacro:box_inertial_with_origin
         mass="100.0"
         x="2"
-        y="0.8"
+        y="0.6"
         z="0.6">
       <origin xyz="-0.05 0 -0.1" />
     </xacro:box_inertial_with_origin>
-    <xacro:box_primitive
+    <xacro:box_primitive_with_origin
         x="2"
-        y="0.8"
-        z="0.6" />
+        y="0.6"
+        z="0.6">
+      <origin xyz="0 0 0.4" />
+    </xacro:box_primitive_with_origin>
   </link>
   <xacro:property
@@ -39,10 +44,13 @@
       front_parent="chassis"
       rear_parent="chassis"
-      front_origin_x="${wheel_track / 2}"
-      rear_origin_x="${-wheel_track / 2}"
-      axle_x="${wheel_track / 2}"
-      gear_x="0.48"
-      socket_x="-0.1"
-      socket_y="0.075"
+      front_origin_x="${wheel_base / 2}"
+      rear_origin_x="${-wheel_base / 2}"
+      axle_x="${wheel_base / 2}"
+      axle_width="${axle_width}"
+      gear_x="${wheel_base / 2 - 0.25}"
+      socket_x="${wheel_base / 2 - 0.25 + 0.08}"
+      socket_y="0.06"
+      rod_x="${wheel_base / 2 - 0.125}"
+      rod_y="${axle_width / 2}"
       z="0" />
   <xacro:wheel
@@ -50,5 +58,5 @@
       parent_link="front_left_axle">
     <origin
-        xyz="0 ${0.156911} 0"
+        xyz="0 ${axle_wheel_offset_y} 0"
         rpy="${pi/2} 0 0" />
   </xacro:wheel>
@@ -57,5 +65,5 @@
       parent_link="front_right_axle">
     <origin
-        xyz="0 ${-0.156911} 0"
+        xyz="0 ${-axle_wheel_offset_y} 0"
         rpy="${pi/2} 0 0" />
   </xacro:wheel>
@@ -64,5 +72,5 @@
       parent_link="rear_left_axle">
     <origin
-        xyz="0 ${0.156911} 0"
+        xyz="0 ${axle_wheel_offset_y} 0"
         rpy="${pi/2} 0 0" />
   </xacro:wheel>
@@ -71,5 +79,5 @@
       parent_link="rear_right_axle">
     <origin
-        xyz="0 ${-0.156911} 0"
+        xyz="0 ${-axle_wheel_offset_y} 0"
         rpy="${pi/2} 0 0" />
   </xacro:wheel>

File: test/models/gazebo_ros_four_wheel_steering_test_vehicle/wheel.urdf.xacro (robot description, xacro)
@@ -9,5 +9,5 @@
       name="drive_max_radps"
       value="6.358" />
-  <xacro:include filename="$(arg xacro_prefix)/urdf/primitives.urdf.xacro" />
+  <xacro:include filename="$(arg gazebo_ros_four_wheel_steering_prefix)/urdf/primitives.urdf.xacro" />
   <xacro:macro
       name="wheel"

File: urdf/axle.urdf.xacro (robot description, xacro)
@@ -4,13 +4,12 @@
       name="gear_size"
       value="0.1" />
-  <xacro:include filename="$(arg xacro_prefix)/urdf/wheel_steered.urdf.xacro" />
-  <xacro:include filename="$(arg xacro_prefix)/urdf/steering_rod.sdf.xacro" />
-  <xacro:include filename="$(arg xacro_prefix)/urdf/primitives.sdf.xacro" />
-  <xacro:include filename="$(arg xacro_prefix)/urdf/inertia_tensors.sdf.xacro" />
+  <xacro:include filename="$(arg gazebo_ros_four_wheel_steering_prefix)/urdf/wheel_steered.urdf.xacro" />
+  <xacro:include filename="$(arg gazebo_ros_four_wheel_steering_prefix)/urdf/steering_rod.sdf.xacro" />
+  <xacro:include filename="$(arg gazebo_ros_four_wheel_steering_prefix)/urdf/primitives.sdf.xacro" />
+  <xacro:include filename="$(arg gazebo_ros_four_wheel_steering_prefix)/urdf/inertia_tensors.sdf.xacro" />
   <!--
   prefix: front, rear
   parent link: should be vehicle chassis
-  is_front: 1 for front, -1 for rear
-  gear_x: offset from axle x position to gear x position, typically negative
+  gear_x: x position of steering gear, assumed y = 0 as in the center of the vehicle
   socket_x: offset from gear to rod socket x position
   socket_y: offset from gear to rod socket y position
@@ -18,16 +17,16 @@
   <xacro:macro
       name="axle"
-      params="prefix parent is_front x gear_x socket_x socket_y z *origin">
+      params="prefix parent x width gear_x socket_x socket_y rod_x rod_y z *origin">
     <xacro:wheel_steered
-        wheel_prefix="${prefix}_left"
+        prefix="${prefix}_left"
         parent_link="${parent}"
         left_right="1">
-      <xacro:insert_block name="origin" />
+      <origin xyz="${x} ${width / 2} ${z}" />
     </xacro:wheel_steered>
     <xacro:wheel_steered
-        wheel_prefix="${prefix}_right"
+        prefix="${prefix}_right"
         parent_link="${parent}"
         left_right="-1">
-      <xacro:insert_block name="origin" />
+      <origin xyz="${x} ${-width / 2} ${z}" />
     </xacro:wheel_steered>
     <!-- SDF-only steering system -->
@@ -35,5 +34,5 @@
       <link name="${prefix}_steering_gear">
         <pose>
-          ${x + gear_x} 0 ${z} 0 0 0
+          ${gear_x} 0 ${z} 0 0 0
         </pose>
         <xacro:sdf_box_inertia
@@ -55,8 +54,8 @@
           <xyz>0 0 1</xyz>
           <limit>
-            <lower>-1.5</lower>
-            <upper>1.5</upper>
-            <effort>2000</effort>
-            <velocity>1.24</velocity>
+            <lower>-0.515446875</lower>
+            <upper>0.515446875</upper>
+            <effort>1000</effort>
+            <velocity>1.1914</velocity>
           </limit>
           <dynamics>
@@ -72,14 +71,18 @@
       </joint>
       <xacro:steering_rod
-          prefix="${prefix}_left"
-          gear_x="${is_front * (x + gear_x)}"
-          rod_x="${is_front * (x + gear_x + socket_x)}"
-          rod_y="${is_front * socket_y}"
+          front_prefix="${prefix}"
+          side_prefix="left"
+          socket_x="${socket_x}"
+          socket_y="${socket_y}"
+          rod_x="${rod_x}"
+          rod_y="${rod_y}"
           z="${z}" />
       <xacro:steering_rod
-          prefix="${prefix}_right"
-          gear_x="${is_front * (x + gear_x)}"
-          rod_x="${is_front * (x + gear_x + socket_x)}"
-          rod_y="${is_front * -socket_y}"
+          front_prefix="${prefix}"
+          side_prefix="right"
+          socket_x="${socket_x}"
+          socket_y="${-socket_y}"
+          rod_x="${rod_x}"
+          rod_y="${-rod_y}"
           z="${z}" />
     </gazebo>

File: urdf/four_wheel_steering.urdf.xacro (robot description, xacro)
@@ -1,16 +1,22 @@
 <?xml version="1.0"?>
 <robot xmlns:xacro="http://ros.org/wiki/xacro">
-  <xacro:include filename="$(arg xacro_prefix)/urdf/axle.urdf.xacro" />
+  <xacro:include filename="$(arg gazebo_ros_four_wheel_steering_prefix)/urdf/axle.urdf.xacro" />
+  <!--
+    front_origin_x and x can in most cases be equal. They are potentially different if in the URDF
+    part of the model, the parent of an axle is not the vehicle center
+  -->
   <xacro:macro
       name="four_wheel_steering"
-      params="front_parent rear_parent front_origin_x rear_origin_x axle_x gear_x socket_x socket_y z">
+      params="front_parent rear_parent front_origin_x rear_origin_x axle_width axle_x gear_x socket_x socket_y rod_x rod_y z">
     <xacro:axle
         prefix="front"
         parent="${front_parent}"
-        is_front="1"
         x="${axle_x}"
+        width="${axle_width}"
         gear_x="${gear_x}"
         socket_x="${socket_x}"
         socket_y="${socket_y}"
+        rod_x="${rod_x}"
+        rod_y="${rod_y}"
         z="${z}">
       <origin xyz="${front_origin_x} 0 ${z}" />
@@ -19,9 +25,11 @@
         prefix="rear"
         parent="${rear_parent}"
-        is_front="-1"
-        x="${axle_x}"
-        gear_x="${gear_x}"
-        socket_x="${socket_x}"
+        x="${-axle_x}"
+        width="${axle_width}"
+        gear_x="${-gear_x}"
+        socket_x="${-socket_x}"
         socket_y="${socket_y}"
+        rod_x="${-rod_x}"
+        rod_y="${rod_y}"
         z="${z}">
       <origin xyz="${rear_origin_x} 0 ${z}" />

File: urdf/primitives.urdf.xacro (robot description, xacro)
@@ -8,4 +8,18 @@
     </visual>
     <collision>
+      <geometry>
+          <box size="${x} ${y} ${z}" />
+      </geometry>
+    </collision>
+  </xacro:macro>
+  <xacro:macro name="box_primitive_with_origin" params="x y z *origin">
+    <visual>
+      <xacro:insert_block name="origin" />
+      <geometry>
+        <box size="${x} ${y} ${z}" />
+      </geometry>
+    </visual>
+    <collision>
+      <xacro:insert_block name="origin" />
       <geometry>
           <box size="${x} ${y} ${z}" />

File: urdf/steering_rod.sdf.xacro (robot description, xacro)
@@ -1,36 +1,36 @@
 <?xml version="1.0"?>
 <sdf xmlns:xacro="http://ros.org/wiki/xacro">
-  <xacro:include filename="$(arg xacro_prefix)/urdf/primitives.sdf.xacro" />
-  <xacro:include filename="$(arg xacro_prefix)/urdf/inertia_tensors.sdf.xacro" />
+  <xacro:include filename="$(arg gazebo_ros_four_wheel_steering_prefix)/urdf/primitives.sdf.xacro" />
+  <xacro:include filename="$(arg gazebo_ros_four_wheel_steering_prefix)/urdf/inertia_tensors.sdf.xacro" />
   <xacro:property name="gear_connector_radius" value="0.05" />
   <xacro:property name="neglectable_mass" value="1" />
-  <xacro:macro name="steering_rod" params="prefix gear_x rod_x rod_y z">
-    <link name="${prefix}_steering_gear">
-      <pose>${gear_x} 0 ${z} 0 0 0</pose>
+  <xacro:macro name="steering_rod" params="front_prefix side_prefix socket_x socket_y rod_x rod_y z">
+    <link name="${front_prefix}_${side_prefix}_steering_gear">
+      <pose>${socket_x} ${socket_y} ${z} 0 0 0</pose>
       <xacro:sdf_sphere_inertia radius="${gear_connector_radius}" mass="${neglectable_mass}" />
       <xacro:sdf_sphere_primitive name="${prefix}" radius="${gear_connector_radius}" />
     </link>
-    <link name="${prefix}_axle_rod_connector">
+    <link name="${front_prefix}_${side_prefix}_axle_rod_connector">
       <pose>${rod_x} ${rod_y} ${z} 0 0 0</pose>
       <xacro:sdf_sphere_inertia radius="${gear_connector_radius}" mass="${neglectable_mass}" />
       <xacro:sdf_sphere_primitive name="${prefix}" radius="${gear_connector_radius}" />
     </link>
-    <joint name="${prefix}_steering_connector" type="revolute">
-      <parent>${prefix}_steering_gear</parent>
-      <child>${prefix}_steering_gear</child>
+    <joint name="${front_prefix}_${side_prefix}_steering_connector" type="revolute">
+      <parent>${front_prefix}_steering_gear</parent>
+      <child>${front_prefix}_${side_prefix}_steering_gear</child>
       <axis>
         <xyz>0 0 1</xyz>
       </axis>
     </joint>
-    <joint name="${prefix}_steering_rod" type="revolute">
-      <parent>${prefix}_steering_gear</parent>
-      <child>${prefix}_axle_rod_connector</child>
+    <joint name="${front_prefix}_${side_prefix}_steering_rod" type="revolute">
+      <parent>${front_prefix}_${side_prefix}_steering_gear</parent>
+      <child>${front_prefix}_${side_prefix}_axle_rod_connector</child>
       <axis>
         <xyz>0 0 1</xyz>
       </axis>
     </joint>
-    <joint name="${prefix}_axle_connection" type="fixed">
-      <parent>${prefix}_axle_rod_connector</parent>
-      <child>${prefix}_axle</child>
+    <joint name="${front_prefix}_${side_prefix}_axle_connection" type="fixed">
+      <parent>${front_prefix}_${side_prefix}_axle_rod_connector</parent>
+      <child>${front_prefix}_${side_prefix}_axle</child>
     </joint>
   </xacro:macro>

File: urdf/wheel_steered.urdf.xacro (robot description, xacro)
@@ -11,6 +11,6 @@
   <xacro:macro
       name="wheel_steered"
-      params="wheel_prefix parent_link left_right *origin">
-    <link name="${wheel_prefix}_axle">
+      params="prefix parent_link left_right *origin">
+    <link name="${prefix}_axle">
       <visual>
         <origin
@@ -36,5 +36,5 @@
     </link>
     <joint
-        name="${wheel_prefix}_kingpin"
+        name="${prefix}_kingpin"
         type="revolute">
       <limit
@@ -45,5 +45,5 @@
       <axis xyz="0 0 1" />
       <parent link="${parent_link}" />
-      <child link="${wheel_prefix}_axle" />
+      <child link="${prefix}_axle" />
       <xacro:insert_block name="origin" />
       <dynamics

Commit message: Controller optimization

File: test/models/gazebo_ros_four_wheel_steering_test_vehicle/model.urdf.xacro (robot description, xacro)
@@ -9,11 +9,11 @@
   <xacro:property
       name="axle_width"
-      value="1.06" />
+      value="1" />
   <xacro:property
       name="axle_wheel_offset_y"
-      value="0.06" />
+      value="0.09" />
   <xacro:property
       name="wheel_base"
-      value="1.1" />
+      value="1.42" />
   <link name="chassis">
     <xacro:box_inertial_with_origin
@@ -41,4 +41,16 @@
       name="mass_wheel"
       value="30.0" />
+  <xacro:property
+    name="steering_gear_triangle_length"
+    value="0.1" />
+  <xacro:property
+    name="socket_x"
+    value="${steering_gear_triangle_length * sin(60 / 180 * pi)}" />
+  <xacro:property
+    name="socket_y"
+    value="${steering_gear_triangle_length * cos(60 / 180 * pi)}" />
+  <xacro:property
+    name="gear_x"
+    value="${wheel_base / 2 - 0.25}" />
   <xacro:four_wheel_steering
       front_parent="chassis"
@@ -48,9 +60,9 @@
       axle_x="${wheel_base / 2}"
       axle_width="${axle_width}"
-      gear_x="${wheel_base / 2 - 0.25}"
-      socket_x="${wheel_base / 2 - 0.25 + 0.08}"
-      socket_y="0.06"
+      gear_x="${gear_x}"
+      socket_x="${gear_x + socket_x}"
+      socket_y="${socket_y}"
       rod_x="${wheel_base / 2 - 0.125}"
-      rod_y="${axle_width / 2}"
+      rod_y="${axle_width / 2 - 0.03}"
       z="0" />
   <xacro:wheel
@@ -93,6 +105,6 @@
       <rear_right_motor_pid_gain>400 0 1</rear_right_motor_pid_gain>
       <rear_left_motor_pid_gain>400 0 1</rear_left_motor_pid_gain>
-      <front_steering_pid_gain>2000 0 2</front_steering_pid_gain>
-      <rear_steering_pid_gain>2000 0 2</rear_steering_pid_gain>
+      <front_steering_pid_gain>4000 100 2</front_steering_pid_gain>
+      <rear_steering_pid_gain>4000 100 2</rear_steering_pid_gain>
     </plugin>
   </gazebo>

Commit message: Validate and output distances on input model

File: test/models/gazebo_ros_four_wheel_steering_test_vehicle/model.urdf.xacro (robot description, xacro)
@@ -58,5 +58,4 @@
       front_origin_x="${wheel_base / 2}"
       rear_origin_x="${-wheel_base / 2}"
-      axle_x="${wheel_base / 2}"
       axle_width="${axle_width}"
       gear_x="${gear_x}"
@@ -65,5 +64,6 @@
       rod_x="${wheel_base / 2 - 0.125}"
       rod_y="${axle_width / 2 - 0.03}"
-      z="0" />
+      z="0"
+      z_sdf="0" />
   <xacro:wheel
       wheel_prefix="front_left"
@@ -98,8 +98,4 @@
         name="gazebo_ros_4ws"
         filename="libgazebo_ros_four_wheel_steering.so">
-      <ros>
-        <namespace>test</namespace>
-      </ros>
-      <latency>0.32</latency>
       <front_right_motor_pid_gain>400 10 1</front_right_motor_pid_gain>
       <front_left_motor_pid_gain>400 10 1</front_left_motor_pid_gain>

File: urdf/axle.urdf.xacro (robot description, xacro)
@@ -17,5 +17,5 @@
   <xacro:macro
       name="axle"
-      params="prefix parent x width gear_x socket_x socket_y rod_x rod_y z *origin">
+      params="prefix parent x width gear_x socket_x socket_y rod_x rod_y z z_sdf">
     <xacro:wheel_steered
         prefix="${prefix}_left"
@@ -34,5 +34,5 @@
       <link name="${prefix}_steering_gear">
         <pose>
-          ${gear_x} 0 ${z} 0 0 0
+          ${gear_x} 0 ${z_sdf} 0 0 0
         </pose>
         <xacro:sdf_box_inertia
@@ -49,11 +49,11 @@
           name="${prefix}_steering"
           type="revolute">
-        <parent>chassis</parent>
+        <parent>${parent}</parent>
         <child>${prefix}_steering_gear</child>
         <axis>
           <xyz>0 0 1</xyz>
           <limit>
-            <lower>-0.515446875</lower>
-            <upper>0.515446875</upper>
+            <lower>-0.61</lower>
+            <upper>0.61</upper>
             <effort>1000</effort>
             <velocity>1.1914</velocity>
@@ -77,5 +77,5 @@
           rod_x="${rod_x}"
           rod_y="${rod_y}"
-          z="${z}" />
+          z="${z_sdf}" />
       <xacro:steering_rod
           front_prefix="${prefix}"
@@ -85,5 +85,5 @@
           rod_x="${rod_x}"
           rod_y="${-rod_y}"
-          z="${z}" />
+          z="${z_sdf}" />
     </gazebo>
   </xacro:macro>

File: urdf/four_wheel_steering.urdf.xacro (robot description, xacro)
@@ -8,9 +8,9 @@
   <xacro:macro
       name="four_wheel_steering"
-      params="front_parent rear_parent front_origin_x rear_origin_x axle_width axle_x gear_x socket_x socket_y rod_x rod_y z">
+      params="front_parent rear_parent front_origin_x rear_origin_x axle_width gear_x socket_x socket_y rod_x rod_y z z_sdf">
     <xacro:axle
         prefix="front"
         parent="${front_parent}"
-        x="${axle_x}"
+        x="${front_origin_x}"
         width="${axle_width}"
         gear_x="${gear_x}"
@@ -19,11 +19,11 @@
         rod_x="${rod_x}"
         rod_y="${rod_y}"
-        z="${z}">
-      <origin xyz="${front_origin_x} 0 ${z}" />
+        z="${z}"
+        z_sdf="${z_sdf}">
     </xacro:axle>
     <xacro:axle
         prefix="rear"
         parent="${rear_parent}"
-        x="${-axle_x}"
+        x="${rear_origin_x}"
         width="${axle_width}"
         gear_x="${-gear_x}"
@@ -32,6 +32,6 @@
         rod_x="${-rod_x}"
         rod_y="${rod_y}"
-        z="${z}">
-      <origin xyz="${rear_origin_x} 0 ${z}" />
+        z="${z}"
+        z_sdf="${z_sdf}">
     </xacro:axle>
   </xacro:macro>
