Commit message: Extend documentation
* introduce gear_transmission_ratio parameter
* add documentation on all parameters and topics
* generalize example

File: test/models/gazebo_ros_four_wheel_steering_test_vehicle/model.urdf.xacro (robot description, xacro)
@@ -42,18 +42,17 @@
       value="30.0" />
   <xacro:property
-    name="steering_gear_triangle_length"
-    value="0.1" />
+      name="steering_gear_triangle_length"
+      value="0.1" />
   <xacro:property
-    name="socket_x"
-    value="${steering_gear_triangle_length * sin(60 / 180 * pi)}" />
+      name="socket_x"
+      value="${steering_gear_triangle_length * sin(60 / 180 * pi)}" />
   <xacro:property
-    name="socket_y"
-    value="${steering_gear_triangle_length * cos(60 / 180 * pi)}" />
+      name="socket_y"
+      value="${steering_gear_triangle_length * cos(60 / 180 * pi)}" />
   <xacro:property
-    name="gear_x"
-    value="${wheel_base / 2 - 0.25}" />
+      name="gear_x"
+      value="${wheel_base / 2 - 0.25}" />
   <xacro:four_wheel_steering
-      front_parent="chassis"
-      rear_parent="chassis"
+      parent="chassis"
       front_origin_x="${wheel_base / 2}"
       rear_origin_x="${-wheel_base / 2}"
@@ -98,4 +97,5 @@
         name="gazebo_ros_4ws"
         filename="libgazebo_ros_four_wheel_steering.so">
+      <steering_gear_transmission_ratio>1.6</steering_gear_transmission_ratio>
       <front_right_motor_pid_gain>400 10 1</front_right_motor_pid_gain>
       <front_left_motor_pid_gain>400 10 1</front_left_motor_pid_gain>

File: test/models/gazebo_ros_four_wheel_steering_test_vehicle/wheel.urdf.xacro (robot description, xacro)
@@ -5,8 +5,8 @@
   <xacro:property
       name="drive_max_nm"
-      value="755" />
+      value="1000.0" />
   <xacro:property
       name="drive_max_radps"
-      value="6.358" />
+      value="6.0" />
   <xacro:include filename="$(arg gazebo_ros_four_wheel_steering_prefix)/urdf/primitives.urdf.xacro" />
   <xacro:macro

File: urdf/axle.urdf.xacro (robot description, xacro)
@@ -54,8 +54,8 @@
           <xyz>0 0 1</xyz>
           <limit>
-            <lower>-0.61</lower>
-            <upper>0.61</upper>
+            <lower>-0.6</lower>
+            <upper>0.6</upper>
             <effort>8000</effort>
-            <velocity>1.1914</velocity>
+            <velocity>1.0</velocity>
           </limit>
           <dynamics>

File: urdf/four_wheel_steering.urdf.xacro (robot description, xacro)
@@ -8,8 +8,8 @@
   <xacro:macro
       name="four_wheel_steering"
-      params="front_parent rear_parent front_origin_x rear_origin_x axle_width gear_x socket_x socket_y rod_x rod_y z z_sdf">
+      params="parent front_origin_x rear_origin_x axle_width gear_x socket_x socket_y rod_x rod_y z z_sdf">
     <xacro:axle
         prefix="front"
-        parent="${front_parent}"
+        parent="${parent}"
         x="${front_origin_x}"
         width="${axle_width}"
@@ -24,5 +24,5 @@
     <xacro:axle
         prefix="rear"
-        parent="${rear_parent}"
+        parent="${parent}"
         x="${rear_origin_x}"
         width="${axle_width}"

File: urdf/primitives.urdf.xacro (robot description, xacro)
@@ -39,3 +39,15 @@
     </collision>
   </xacro:macro>
+  <xacro:macro name="sphere_primitive" params="radius">
+    <visual>
+      <geometry>
+        <sphere radius="${radius}" />
+      </geometry>
+    </visual>
+    <collision>
+      <geometry>
+        <sphere radius="${radius}" />
+      </geometry>
+    </collision>
+  </xacro:macro>
 </robot>

File: urdf/wheel_steered.urdf.xacro (robot description, xacro)
@@ -3,6 +3,7 @@
     xmlns:xacro="http://ros.org/wiki/xacro"
     name="wheel_steered">
+  <xacro:include filename="$(arg gazebo_ros_four_wheel_steering_prefix)/urdf/primitives.urdf.xacro" />
   <xacro:property
-      name="steering_mass_radius"
+      name="axle_link_radius"
       value="0.1" />
   <xacro:property
@@ -13,22 +14,7 @@
       params="prefix parent_link left_right *origin">
     <link name="${prefix}_axle">
-      <visual>
-        <origin
-            xyz="0 0 0"
-            rpy="${pi/2} 0 0" />
-        <geometry>
-          <mesh filename="package://metron_p48_description/media/models/wheels/motor.dae" />
-        </geometry>
-        <material name="gray">
-          <color rgba="0.4 0.4 0.4 1.0" />
-        </material>
-      </visual>
-      <collision>
-        <geometry>
-          <sphere radius="0.2" />
-        </geometry>
-      </collision>
+      <xacro:sphere_primitive radius="${axle_link_radius}" />
       <xacro:sphere_inertial_with_origin
-          radius="${steering_mass_radius}"
+          radius="${axle_link_radius}"
           mass="${steering_link_mass}">
         <origin xyz="0 ${-0.1 * left_right} 0" />
@@ -39,8 +25,8 @@
         type="revolute">
       <limit
-          lower="-0.6109"
-          upper="0.6109"
+          lower="-0.6"
+          upper="0.6"
           effort="4000"
-          velocity="1.4" />
+          velocity="1.0" />
       <axis xyz="0 0 1" />
       <parent link="${parent_link}" />
