Commit message: Plausible steering joint configuration

File: urdf/axle.urdf.xacro (robot description, xacro)
@@ -56,10 +56,10 @@
             <lower>-0.61</lower>
             <upper>0.61</upper>
-            <effort>1000</effort>
+            <effort>8000</effort>
             <velocity>1.1914</velocity>
           </limit>
           <dynamics>
-            <damping>1</damping>
-            <friction>2</friction>
+            <damping>0</damping>
+            <friction>5</friction>
           </dynamics>
         </axis>

File: urdf/wheel_steered.urdf.xacro (robot description, xacro)
@@ -41,5 +41,5 @@
           lower="-0.6109"
           upper="0.6109"
-          effort="1000"
+          effort="4000"
           velocity="1.4" />
       <axis xyz="0 0 1" />
@@ -47,7 +47,5 @@
       <child link="${prefix}_axle" />
       <xacro:insert_block name="origin" />
-      <dynamics
-          damping="1.0"
-          friction="0" />
+      <dynamics friction="0" />
       <gazebo>
         <physics>
